Commit message: 控制不确定性+感知不确定性+速度规划(春节前版本)

File: src/gpir/planning_core/3d_model/3d_model.xacro (robot description, xacro)
@@ -3,7 +3,9 @@
   <link name="ego_vehicle2d">
     <visual>
-      <origin xyz="0 0 1.0" rpy="0 0 1.5707963267948966"/>
+      <!-- <origin xyz="0 0 1.0" rpy="0 0 1.5707963267948966"/> -->
+      <origin xyz="0 0 0" rpy="1.570796326794896 0 3.1415926"/>
       <geometry>
-        <mesh filename="package://planning_core/3d_model/model3/model3.dae" scale="1.0 1.0 1.0"/>
+        <!-- <mesh filename="package://planning_core/3d_model/model3/model3.dae" scale="1.0 1.0 1.0"/> -->
+        <mesh filename="package://planning_core/3d_model/lexus/lexus.dae" scale="1.0 1.0 1.0"/>
       </geometry>
     </visual>

Commit message: 4o版本的更改代价函数

File: src/gpir/planning_core/3d_model/3d_model.xacro (robot description, xacro)
@@ -3,9 +3,9 @@
   <link name="ego_vehicle2d">
     <visual>
-      <!-- <origin xyz="0 0 1.0" rpy="0 0 1.5707963267948966"/> -->
-      <origin xyz="0 0 0" rpy="1.570796326794896 0 3.1415926"/>
+      <origin xyz="0 0 1.0" rpy="0 0 1.5707963267948966"/>
+      <!-- <origin xyz="0 0 0" rpy="1.570796326794896 0 3.1415926"/> -->
       <geometry>
-        <!-- <mesh filename="package://planning_core/3d_model/model3/model3.dae" scale="1.0 1.0 1.0"/> -->
-        <mesh filename="package://planning_core/3d_model/lexus/lexus.dae" scale="1.0 1.0 1.0"/>
+        <mesh filename="package://planning_core/3d_model/model3/model3.dae" scale="1.0 1.0 1.0"/>
+        <!-- <mesh filename="package://planning_core/3d_model/lexus/lexus.dae" scale="1.0 1.0 1.0"/> -->
       </geometry>
     </visual>
